File: pathfinderKey-Cuts.kicad_pcb (KiCad board)
At the start: 2 copper layers, 81 x 71 mm, 13 parts, among them SW1 SW_Push, SW2 SW_Push, SW3 SW_Push, SW4 SW_Push, U1 XIAO-RP2040-DIP

Commit message: Add files via upload
Routing:
- net GND: track 142.3 -> 148.6 mm
- net LED1: track 151.4 -> 149.2 mm
- net LED3: track 74.7 -> 72.4 mm
- net button1: track 114.2 -> 116.0 mm
- net button4: track 55.6 -> 54.5 mm
